File: kicad/main.kicad_pcb (KiCad board)
At the start: 2 copper layers, 150 x 100 mm, 96 parts, among them J1 Screw_Terminal_01x10, J2 Screw_Terminal_01x02, J3 Conn_01x03, J4 Conn_01x03, Q1 IRF540N, Q2 IRF540N, Q3 IRF540N, Q4 IRF540N, Q5 IRF540N, SW2 Switch_All, SW3 Switch1, SW4 Switch2, SW5 Switch3, SW6 Switch4, SW7 Switch5, U1 L7805, U2 ATmega328P-PU, U3 PC817, U4 PC817, U5 PC817, U6 PC817, U7 PC817, Y1 16mHz

Commit message: update
Parts:
- BTN1: footprint local_footprint:JST_VH_B2P-VH_1x02_P3.96mm_Vertical -> Button_Switch_SMD:SW_SPST_PTS645
- moved JP1 18.5 mm to (67.8, 120.3)
- moved BTN1 5.68 mm to (115.8, 126.6), turned to 0 degrees
Routing:
- net +12V: track 375.9 -> 366.4 mm
- net /RESET: track 68.3 -> 72.9 mm
- net GNDREF: track 35.6 -> 40.0 mm, vias 0 -> 5
- net GNDS: vias 0 -> 12
Other:
- board text added: "2021/11/13"
- board text removed: "2021/10/03"
